Commit message: edit axis for adjusting solidworks model

File: mdl_description/urdf/mdl_description.xacro (robot description, xacro)
@@ -22,17 +22,17 @@
           rpy="0 0 0" />
         <geometry>
-          <mesh filename="package://mdl_description/meshes/Link_1.dae" />
-        </geometry>
-        <material name="red">
-          <color rgba="1.0 0.0 0.0 2.0"/>
-        </material>
-      </visual>
-      <collision>
-        <origin
-          xyz="0 0 0"
-          rpy="0 0 0" />
-        <geometry>
-          <mesh
-            filename="package://mdl_description/meshes/Link_1.dae" />
+          <mesh filename="package://mdl_description/meshes/Link_1.STL" />
+        </geometry>
+        <material name="red">
+          <color rgba="1.0 0.0 0.0 2.0"/>
+        </material>
+      </visual>
+      <collision>
+        <origin
+          xyz="0 0 0"
+          rpy="0 0 0" />
+        <geometry>
+          <mesh
+            filename="package://mdl_description/meshes/Link_1.STL" />
         </geometry>
       </collision>
@@ -60,17 +60,17 @@
         <geometry>
           <mesh
-            filename="package://mdl_description/meshes/Link_2.dae" />
-        </geometry>
-        <material name="red">
-          <color rgba="1.0 0.0 0.0 2.0"/>
-        </material>
-      </visual>
-      <collision>
-        <origin
-          xyz="0 0 0"
-          rpy="0 0 0" />
-        <geometry>
-          <mesh
-            filename="package://mdl_description/meshes/Link_2.dae" />
+            filename="package://mdl_description/meshes/Link_2.STL" />
+        </geometry>
+        <material name="red">
+          <color rgba="1.0 0.0 0.0 2.0"/>
+        </material>
+      </visual>
+      <collision>
+        <origin
+          xyz="0 0 0"
+          rpy="0 0 0" />
+        <geometry>
+          <mesh
+            filename="package://mdl_description/meshes/Link_2.STL" />
         </geometry>
       </collision>
@@ -111,17 +111,17 @@
         <geometry>
           <mesh
-            filename="package://mdl_description/meshes/Link_3.dae" />
-        </geometry>
-        <material name="red">
-          <color rgba="1.0 0.0 0.0 2.0"/>
-        </material>
-      </visual>
-      <collision>
-        <origin
-          xyz="0 0 0"
-          rpy="0 0 0" />
-        <geometry>
-          <mesh
-            filename="package://mdl_description/meshes/Link_3.dae" />
+            filename="package://mdl_description/meshes/Link_3.STL" />
+        </geometry>
+        <material name="red">
+          <color rgba="1.0 0.0 0.0 2.0"/>
+        </material>
+      </visual>
+      <collision>
+        <origin
+          xyz="0 0 0"
+          rpy="0 0 0" />
+        <geometry>
+          <mesh
+            filename="package://mdl_description/meshes/Link_3.STL" />
         </geometry>
       </collision>
@@ -132,5 +132,5 @@
       <origin
         xyz="0 0 0.1"
-        rpy="1.5708 -1.5708 0" />
+        rpy="-1.5708 -1.5708 0" />
       <parent
         link="Link_2" />
@@ -162,17 +162,17 @@
         <geometry>
           <mesh
-            filename="package://mdl_description/meshes/Link_4.dae" />
-        </geometry>
-        <material name="red">
-          <color rgba="1.0 0.0 0.0 2.0"/>
-        </material>
-      </visual>
-      <collision>
-        <origin
-          xyz="0 0 0"
-          rpy="0 0 0" />
-        <geometry>
-          <mesh
-            filename="package://mdl_description/meshes/Link_4.dae" />
+            filename="package://mdl_description/meshes/Link_4.STL" />
+        </geometry>
+        <material name="red">
+          <color rgba="1.0 0.0 0.0 2.0"/>
+        </material>
+      </visual>
+      <collision>
+        <origin
+          xyz="0 0 0"
+          rpy="0 0 0" />
+        <geometry>
+          <mesh
+            filename="package://mdl_description/meshes/Link_4.STL" />
         </geometry>
       </collision>
@@ -189,5 +189,5 @@
         link="Link_4" />
       <axis
-        xyz="0 0 -1" />
+        xyz="0 0 1" />
     </joint>
     <link
@@ -213,17 +213,17 @@
         <geometry>
           <mesh
-            filename="package://mdl_description/meshes/Link_5.dae" />
-        </geometry>
-        <material name="red">
-          <color rgba="1.0 0.0 0.0 2.0"/>
-        </material>
-      </visual>
-      <collision>
-        <origin
-          xyz="0 0 0"
-          rpy="0 0 0" />
-        <geometry>
-          <mesh
-            filename="package://mdl_description/meshes/Link_5.dae" />
+            filename="package://mdl_description/meshes/Link_5.STL" />
+        </geometry>
+        <material name="red">
+          <color rgba="1.0 0.0 0.0 2.0"/>
+        </material>
+      </visual>
+      <collision>
+        <origin
+          xyz="0 0 0"
+          rpy="0 0 0" />
+        <geometry>
+          <mesh
+            filename="package://mdl_description/meshes/Link_5.STL" />
         </geometry>
       </collision>
@@ -240,5 +240,5 @@
         link="Link_5" />
       <axis
-        xyz="0 0 -1" />
+        xyz="0 0 1" />
     </joint>
     <link
@@ -264,17 +264,17 @@
         <geometry>
           <mesh
-            filename="package://mdl_description/meshes/Link_6.dae" />
-        </geometry>
-        <material name="red">
-          <color rgba="1.0 0.0 0.0 2.0"/>
-        </material>
-      </visual>
-      <collision>
-        <origin
-          xyz="0 0 0"
-          rpy="0 0 0" />
-        <geometry>
-          <mesh
-            filename="package://mdl_description/meshes/Link_6.dae" />
+            filename="package://mdl_description/meshes/Link_6.STL" />
+        </geometry>
+        <material name="red">
+          <color rgba="1.0 0.0 0.0 2.0"/>
+        </material>
+      </visual>
+      <collision>
+        <origin
+          xyz="0 0 0"
+          rpy="0 0 0" />
+        <geometry>
+          <mesh
+            filename="package://mdl_description/meshes/Link_6.STL" />
         </geometry>
       </collision>
@@ -291,5 +291,5 @@
         link="Link_6" />
       <axis
-        xyz="0 0 -1" />
+        xyz="0 0 1" />
     </joint>
   </xacro:macro>
