Commit message: change virtual joint setting from fixed to float

File: mdl_moveit_config/config/simple_5dof_robot.ros2_control.xacro (robot description, xacro)
@@ -8,4 +8,11 @@
                 <plugin>mock_components/GenericSystem</plugin>
             </hardware>
+            <joint name="vitrual_joint_EE_1">
+                <command_interface name="position"/>
+                <state_interface name="position">
+                  <param name="initial_value">${initial_positions['vitrual_joint_EE_1']}</param>
+                </state_interface>
+                <state_interface name="velocity"/>
+            </joint>
             <joint name="Joint_1">
                 <command_interface name="position"/>

Commit message: Marge moveit_config_floating

File: mdl_moveit_config/config/simple_5dof_robot.ros2_control.xacro (robot description, xacro)
@@ -8,11 +8,4 @@
                 <plugin>mock_components/GenericSystem</plugin>
             </hardware>
-            <joint name="vitrual_joint_EE_1">
-                <command_interface name="position"/>
-                <state_interface name="position">
-                  <param name="initial_value">${initial_positions['vitrual_joint_EE_1']}</param>
-                </state_interface>
-                <state_interface name="velocity"/>
-            </joint>
             <joint name="Joint_1">
                 <command_interface name="position"/>
