Commit message: update display_cube.launch.py

File: mdl_cube_description/urdf/mdl_cube.xacro (robot description, xacro)
@@ -5,12 +5,14 @@
 <xacro:include filename="$(find mdl_cube_description)/urdf/mdl_cube_description.xacro" />
 <xacro:base_macro/>
-<xacro:mdl_cube_description prefix="mdl_cube_00" parent="base_link" pos_xyz="0.00 0.00 0.06" mdl_cube_color="color_0"/>
-<xacro:mdl_cube_description prefix="mdl_cube_01" parent="base_link" pos_xyz="0.00 0.00 0.18" mdl_cube_color="color_2"/>
-<xacro:mdl_cube_description prefix="mdl_cube_02" parent="base_link" pos_xyz="0.00 0.00 0.30" mdl_cube_color="color_4"/>
-<xacro:mdl_cube_description prefix="mdl_cube_03" parent="base_link" pos_xyz="0.12 0.00 0.06" mdl_cube_color="color_6"/>
-<xacro:mdl_cube_description prefix="mdl_cube_04" parent="base_link" pos_xyz="0.12 0.00 0.18" mdl_cube_color="color_8"/>
-<xacro:mdl_cube_description prefix="mdl_cube_05" parent="base_link" pos_xyz="0.12 0.00 0.30" mdl_cube_color="color_10"/>
-<xacro:mdl_cube_description prefix="mdl_cube_06" parent="base_link" pos_xyz="0.24 0.00 0.06" mdl_cube_color="color_12"/>
-<xacro:mdl_cube_description prefix="mdl_cube_07" parent="base_link" pos_xyz="0.24 0.00 0.18" mdl_cube_color="color_14"/>
-<xacro:mdl_cube_description prefix="mdl_cube_08" parent="base_link" pos_xyz="0.24 0.00 0.30" mdl_cube_color="color_16"/>
+<!-- To switch initial assembly configuration-->
+<xacro:arg name="grid_6" default="false" />
+<!-- grid_6-->
+<xacro:if value="$(arg grid_6)">
+  <xacro:mdl_cube_description prefix="mdl_cube_00" parent="base_link" pos_xyz="0.00 0.00 0.06" rpy="0 0 0" body_color="color_0" f0_color="color_0" f1_color="color_0" f2_color="color_0" f3_color="color_0" f4_color="color_0" f5_color="color_0"/>
+  <xacro:mdl_cube_description prefix="mdl_cube_01" parent="base_link" pos_xyz="0.00 0.00 0.18" rpy="0 0 0" body_color="color_0" f0_color="color_0" f1_color="color_0" f2_color="color_0" f3_color="color_0" f4_color="color_0" f5_color="color_0"/>
+  <xacro:mdl_cube_description prefix="mdl_cube_02" parent="base_link" pos_xyz="0.00 0.00 0.30" rpy="0 0 0" body_color="color_0" f0_color="color_0" f1_color="color_0" f2_color="color_0" f3_color="color_0" f4_color="color_0" f5_color="color_0"/>
+  <xacro:mdl_cube_description prefix="mdl_cube_03" parent="base_link" pos_xyz="0.12 0.00 0.06" rpy="0 0 0" body_color="color_0" f0_color="color_0" f1_color="color_0" f2_color="color_0" f3_color="color_0" f4_color="color_0" f5_color="color_0"/>
+  <xacro:mdl_cube_description prefix="mdl_cube_04" parent="base_link" pos_xyz="0.12 0.00 0.18" rpy="0 0 0" body_color="color_0" f0_color="color_0" f1_color="color_0" f2_color="color_0" f3_color="color_0" f4_color="color_0" f5_color="color_0"/>
+  <xacro:mdl_cube_description prefix="mdl_cube_05" parent="base_link" pos_xyz="0.12 0.00 0.30" rpy="0 0 0" body_color="color_0" f0_color="color_0" f1_color="color_0" f2_color="color_0" f3_color="color_0" f4_color="color_0" f5_color="color_0"/>
+</xacro:if>
 </robot>

File: mdl_cube_description/urdf/mdl_cube_description.xacro (robot description, xacro)
@@ -2,22 +2,108 @@
 <robot name="modular_cube"  xmlns:xacro="http://www.ros.org/wiki/xacro" >
   <!-- <xacro:macro name="mdl_cube_description" params="color_0"> -->
-  <xacro:macro name="mdl_cube_description" params="prefix parent pos_xyz mdl_cube_color">
-    <joint name="${prefix}_body_joint" type="fixed">
-      <origin
-        rpy="0 0 0"
-        xyz="${pos_xyz}"/>
+  <xacro:macro name="mdl_cube_description" params="prefix parent pos_xyz rpy body_color f0_color f1_color f2_color f3_color f4_color f5_color">
+    <link name="${prefix}_body_link">
+      <visual>
+        <origin xyz="0 0 0" rpy="0 0 0"/>
+        <geometry>
+          <box size="0.11 0.11 0.11"/>
+        </geometry>
+        <material name="${body_color}"/>
+      </visual>
+      <inertial>
+        <origin xyz="0 0 0" rpy="0 0 0"/>
+        <mass value="1"/>
+        <inertia ixx="0" ixy="0" ixz="0" iyy="0" iyz="0" izz="0"/>
+      </inertial>
+    </link>
+    <joint name="${prefix}_base_joint" type="fixed">
+      <origin xyz="${pos_xyz}" rpy="${rpy}"/>
       <parent link="${parent}"/>
       <child link="${prefix}_body_link"/>
     </joint>
-    <link name="${prefix}_body_link">
+    <link name="${prefix}_face_0_link">
       <visual>
+        <origin xyz="0 0 0" rpy="0 0 0"/>
         <geometry>
-          <box size="0.12 0.12 0.12"/>
+          <box size="-0.01 0.11 0.11"/>
         </geometry>
-        <origin xyz="0 0 0" rpy="0 0 0"/>
-        <material name="${mdl_cube_color}">
-        </material>
+        <material name="${f0_color}"/>
       </visual>
     </link>
+    <joint name="${prefix}_face_0_joint" type="fixed">
+      <origin xyz="0.06 0 0" rpy="0 0 0"/>
+      <parent link="${prefix}_body_link"/>
+      <child link="${prefix}_face_0_link"/>
+    </joint>
+    <link name="${prefix}_face_1_link">
+      <visual>
+        <origin xyz="0 0 0" rpy="0 0 0"/>
+        <geometry>
+          <box size="0.11 -0.01 0.11"/>
+        </geometry>
+        <material name="${f1_color}"/>
+      </visual>
+    </link>
+    <joint name="${prefix}_face_1_joint" type="fixed">
+      <origin xyz="0 0.06 0" rpy="0 0 0"/>
+      <parent link="${prefix}_body_link"/>
+      <child link="${prefix}_face_1_link"/>
+    </joint>
+    <link name="${prefix}_face_2_link">
+      <visual>
+        <origin xyz="0 0 0" rpy="0 0 0"/>
+        <geometry>
+          <box size="0.11 0.11 -0.01"/>
+        </geometry>
+        <material name="${f2_color}"/>
+      </visual>
+    </link>
+    <joint name="${prefix}_face_2_joint" type="fixed">
+      <origin xyz="0 0 0.06" rpy="0 0 0"/>
+      <parent link="${prefix}_body_link"/>
+      <child link="${prefix}_face_2_link"/>
+    </joint>
+    <link name="${prefix}_face_3_link">
+      <visual>
+        <origin xyz="0 0 0" rpy="0 0 0"/>
+        <geometry>
+          <box size="0.01 0.11 0.11"/>
+        </geometry>
+        <material name="${f3_color}"/>
+      </visual>
+    </link>
+    <joint name="${prefix}_face_3_joint" type="fixed">
+      <origin xyz="-0.06 0 0" rpy="0 0 0"/>
+      <parent link="${prefix}_body_link"/>
+      <child link="${prefix}_face_3_link"/>
+    </joint>
+    <link name="${prefix}_face_4_link">
+      <visual>
+        <origin xyz="0 0 0" rpy="0 0 0"/>
+        <geometry>
+          <box size="0.11 0.01 0.11"/>
+        </geometry>
+        <material name="${f4_color}"/>
+      </visual>
+    </link>
+    <joint name="${prefix}_face_4_joint" type="fixed">
+      <origin xyz="0 -0.06 0" rpy="0 0 0"/>
+      <parent link="${prefix}_body_link"/>
+      <child link="${prefix}_face_4_link"/>
+    </joint>
+    <link name="${prefix}_face_5_link">
+      <visual>
+        <origin xyz="0 0 0" rpy="0 0 0"/>
+        <geometry>
+          <box size="0.11 0.11 0.01"/>
+        </geometry>
+        <material name="${f5_color}"/>
+      </visual>
+    </link>
+    <joint name="${prefix}_face_5_joint" type="fixed">
+      <origin xyz="0 0 -0.06" rpy="0 0 0"/>
+      <parent link="${prefix}_body_link"/>
+      <child link="${prefix}_face_5_link"/>
+    </joint>
   </xacro:macro>
 </robot>
